Commit message: spawned the URDF in gazebo harmonic

File: champ_description/urdf/champ.urdf (robot description, URDF)
Before this commit: robot champ, 29 links, 28 joints
Links:
- link base_link: geometry collision mesh filename=file:///home/sunbeam/projects/quadruped/install/champ_descr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 scale=0.001 0.001 0.001; visual mesh filename=file:///home/sunbeam/projects/quadruped/install/champ_descr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 scale=0.001 0.001 0.001
- link camera_link: geometry collision mesh filename=file:///home/sunbeam/projects/quadruped/install/champ_descr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; visual mesh filename=file:///home/sunbeam/projects/quadruped/install/champ_descr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
- link hokuyo_frame: geometry collision box size=0.058 0.058 0.087; visual mesh filename=file:///home/sunbeam/projects/quadruped/install/champ_descr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
- link lf_hip_link: geometry collision mesh filename=file:///home/sunbeam/projects/quadruped/install/champ_descr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 scale=0.001 0.001 0.001; visual mesh filename=file:///home/sunbeam/projects/quadruped/install/champ_descr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 scale=0.001 0.001 0.001
- link lf_lower_leg_link: geometry collision mesh filename=file:///home/sunbeam/projects/quadruped/install/champ_descr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 scale=0.001 0.001 0.001; visual mesh filename=file:///home/sunbeam/projects/quadruped/install/champ_descr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 scale=0.001 0.001 0.001
- link lf_upper_leg_link: geometry collision mesh filename=file:///home/sunbeam/projects/quadruped/install/champ_descr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 scale=0.001 0.001 0.001; visual mesh filename=file:///home/sunbeam/projects/quadruped/install/champ_descr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 scale=0.001 0.001 0.001
- link lh_hip_link: geometry collision mesh filename=file:///home/sunbeam/projects/quadruped/install/champ_descr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 scale=0.001 0.001 0.001; visual mesh filename=file:///home/sunbeam/projects/quadruped/install/champ_descr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 scale=0.001 0.001 0.001
- link lh_lower_leg_link: geometry collision mesh filename=file:///home/sunbeam/projects/quadruped/install/champ_descr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 scale=0.001 0.001 0.001; visual mesh filename=file:///home/sunbeam/projects/quadruped/install/champ_descr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 scale=0.001 0.001 0.001
- link lh_upper_leg_link: geometry collision mesh filename=file:///home/sunbeam/projects/quadruped/install/champ_descr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 scale=0.001 0.001 0.001; visual mesh filename=file:///home/sunbeam/projects/quadruped/install/champ_descr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 scale=0.001 0.001 0.001
- link rf_hip_link: geometry collision mesh filename=file:///home/sunbeam/projects/quadruped/install/champ_descr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 scale=0.001 0.001 0.001; visual mesh filename=file:///home/sunbeam/projects/quadruped/install/champ_descr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 scale=0.001 0.001 0.001
- link rf_lower_leg_link: geometry collision mesh filename=file:///home/sunbeam/projects/quadruped/install/champ_descr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 scale=0.001 0.001 0.001; visual mesh filename=file:///home/sunbeam/projects/quadruped/install/champ_descr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 scale=0.001 0.001 0.001
- link rf_upper_leg_link: geometry collision mesh filename=file:///home/sunbeam/projects/quadruped/install/champ_descr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 scale=0.001 0.001 0.001; visual mesh filename=file:///home/sunbeam/projects/quadruped/install/champ_descr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 scale=0.001 0.001 0.001
- link rh_hip_link: geometry collision mesh filename=file:///home/sunbeam/projects/quadruped/install/champ_descr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 scale=0.001 0.001 0.001; visual mesh filename=file:///home/sunbeam/projects/quadruped/install/champ_descr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 scale=0.001 0.001 0.001
- link rh_lower_leg_link: geometry collision mesh filename=file:///home/sunbeam/projects/quadruped/install/champ_descr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 scale=0.001 0.001 0.001; visual mesh filename=file:///home/sunbeam/projects/quadruped/install/champ_descr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 scale=0.001 0.001 0.001
- link rh_upper_leg_link: geometry collision mesh filename=file:///home/sunbeam/projects/quadruped/install/champ_descr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 scale=0.001 0.001 0.001; visual mesh filename=file:///home/sunbeam/projects/quadruped/install/champ_descr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 scale=0.001 0.001 0.001

File: champ_description/urdf/champ.urdf.xacro (robot description, xacro)
@@ -41,5 +41,5 @@
     </gazebo>
     <xacro:include filename="$(find champ_description)/urdf/leg.urdf.xacro" />
-    <xacro:include filename="$(find champ_description)/urdf/accessories.urdf.xacro" />
+    <!-- <xacro:include filename="$(find champ_description)/urdf/accessories.urdf.xacro" /> -->
     <xacro:accessories
         base_name="base_link"
@@ -51,5 +51,5 @@
     <xacro:champ_leg leg="rf"/>
     <xacro:champ_leg leg="rh"/>
-    <gazebo>
+    <!-- <gazebo>
       <plugin name="p3d_base_controller" filename="libgazebo_ros_p3d.so">
         <ros>
@@ -68,4 +68,4 @@
         <parameters>$(find champ_gazebo)/config/ros_control.yaml</parameters>
       </plugin>
-    </gazebo>
+    </gazebo> -->
 </robot>
